Commit message: feat: add .urdf file for visualization of the simulation using RViz

File: src/cartpole_sim/urdf/cartpole.urdf.xacro (robot description, xacro)
@@ -1,5 +1,40 @@
 <?xml version="1.0"?>
 <robot name="cartpole">
+    <link name="world">
+    </link>
     <link name="cart">
+        <visual>
+            <geometry>
+                <box size="0.5 0.2 0.1"/>
+            </geometry>
+        </visual>
     </link>
+    <link name="pendulum">
+        <visual>
+            <geometry>
+                <cylinder length="1.0" radius="0.01"/>
+            </geometry>
+            <origin xyz="0 0 0.5"/>
+        </visual>
+        <visual>
+            <geometry>
+                <cylinder length="0.1" radius="0.2"/>
+            </geometry>
+            <origin xyz="0 0 1"/>
+        </visual>
+    </link>
+    <!-- Joints of the system -->
+    <joint name="cart_joint" type="prismatic">
+        <parent link="world"/>
+        <child link="cart"/>
+        <origin xyz="0 0 0"/>
+        <axis xyz="1 0 0"/>
+        <limit effort="1000.0" lower="-2.0" upper="2.0" velocity="100"/>
+    </joint>
+    <joint name="pendulum_joint" type="continuous">
+        <parent link="cart"/>
+        <child link="pendulum"/>
+        <origin xyz="0 0 0.05" rpy="0 0 0"/>
+        <axis xyz="0 1 0"/>
+    </joint>
 </robot>

Commit message: feat: implement a launch.py file for easier simulation launching, rviz config file for instant visualization when launching the simulation and update the documentation with the new integrations

File: src/cartpole_sim/urdf/cartpole.urdf.xacro (robot description, xacro)
@@ -19,7 +19,7 @@
         <visual>
             <geometry>
-                <cylinder length="0.1" radius="0.2"/>
+                <cylinder length="0.1" radius="0.05"/>
             </geometry>
-            <origin xyz="0 0 1"/>
+            <origin xyz="0 0 1" rpy="1.57 0 0"/>
         </visual>
     </link>
